Commit message: refresh

File: robotiq_2f_85_description/urdf/robotiq_2F_85.xacro (robot description, xacro)
@@ -1,27 +1,33 @@
 <?xml version="1.0"?>
-<robot xmlns:xacro="http://ros.org/wiki/xacro">
-  <xacro:macro name="robotiq_arg2f_base_link" params="prefix">
-    <link name="${prefix}robotiq_arg2f_base_link">
-      <inertial>
-        <origin xyz="8.625E-08 -4.6583E-06 0.03145" rpy="0 0 0" />
-        <mass value="0.22652" />
-        <inertia ixx="0.00020005" ixy="-4.2442E-10" ixz="-2.9069E-10" iyy="0.00017832" iyz="-3.4402E-08" izz="0.00013478" />
-      </inertial>
-      <visual>
-        <origin xyz="0 0 0" rpy="0 0 0" />
-        <geometry>
-          <mesh filename="package://robotiq_2f_85_description/meshes/visual/robotiq_arg2f_85_base_link.dae" scale="0.001 0.001 0.001"/>
-        </geometry>
-        <material name="">
-          <color rgba="0.1 0.1 0.1 1" />
-        </material>
-      </visual>
-      <collision>
-        <origin xyz="0 0 0" rpy="0 0 0" />
-        <geometry>
-           <mesh filename="package://robotiq_2f_85_description/meshes/collision/robotiq_arg2f_base_link.stl" />
-        </geometry>
-      </collision>
-    </link>
-  </xacro:macro>
+<robot name="robotiq_arg2f_85" xmlns:xacro="http://ros.org/wiki/xacro">
+  <xacro:include filename="$(find robotiq_2f_85_description)/urdf/robotiq_arg2f_85_model_macro.xacro" />
+  <xacro:robotiq_arg2f_85 prefix=""/>
+	<link name="world"/>
+  <link name="coupling_link">
+    <visual>
+      <origin xyz="0 0 0.007" rpy="0 0 ${pi/2}" />
+      <geometry>
+        <mesh filename="package://robotiq_2f_85_description/meshes/visual/robotiq_gripper_coupling.stl" scale="0.001 0.001 0.001"/>
+      </geometry>
+      <material name="">
+        <color rgba="0.1 0.1 0.1 1" />
+      </material>
+    </visual>
+    <collision>
+      <origin xyz="0 0 0" rpy="0 0 0" />
+      <geometry>
+          <mesh filename="package://robotiq_2f_85_description/meshes/visual/robotiq_gripper_coupling.stl" />
+      </geometry>
+    </collision>
+  </link>
+	<joint name="world" type="fixed">
+		<parent link="world"/>
+		<child link="coupling_link"/>
+		<origin xyz="0 0 0" rpy="0 0 0"/>
+	</joint>
+  <joint name="coupling_joint" type="fixed">
+    <origin xyz="0 0 0.011" rpy="0 0 0"/>
+    <parent link="coupling_link" />
+    <child link="robotiq_arg2f_base_link" />
+  </joint>
 </robot>

File: robotiq_2f_85_description/urdf/robotiq_arg2f_85_model_macro.xacro (robot description, xacro)
@@ -1,6 +1,6 @@
 <?xml version="1.0"?>
 <robot xmlns:xacro="http://ros.org/wiki/xacro">
+  <xacro:include filename="$(find robotiq_2f_85_description)/urdf/robotiq_arg2f.xacro" />
   <xacro:include filename="$(find robotiq_2f_85_description)/urdf/robotiq_arg2f_transmission.xacro" />
-  <xacro:include filename="$(find robotiq_2f_85_description)/urdf/robotiq_arg2f.xacro" />
   <xacro:macro name="outer_knuckle" params="prefix fingerprefix stroke">
     <link name="${prefix}${fingerprefix}_outer_knuckle">

Commit message: refresh

File: robotiq_2f_85_description/urdf/robotiq_2F_85.xacro (robot description, xacro)
@@ -3,5 +3,4 @@
   <xacro:include filename="$(find robotiq_2f_85_description)/urdf/robotiq_arg2f_85_model_macro.xacro" />
   <xacro:robotiq_arg2f_85 prefix=""/>
-	<link name="world"/>
   <link name="coupling_link">
     <visual>
@@ -21,9 +20,4 @@
     </collision>
   </link>
-	<joint name="world" type="fixed">
-		<parent link="world"/>
-		<child link="coupling_link"/>
-		<origin xyz="0 0 0" rpy="0 0 0"/>
-	</joint>
   <joint name="coupling_joint" type="fixed">
     <origin xyz="0 0 0.011" rpy="0 0 0"/>

Commit message: update

File: robotiq_2f_85_description/urdf/robotiq_2F_85.xacro (robot description, xacro)
@@ -1,4 +1,4 @@
 <?xml version="1.0"?>
-<robot name="robotiq_arg2f_85" xmlns:xacro="http://ros.org/wiki/xacro">
+<robot name="robotiq_arg2f_85_model" xmlns:xacro="http://ros.org/wiki/xacro">
   <xacro:include filename="$(find robotiq_2f_85_description)/urdf/robotiq_arg2f_85_model_macro.xacro" />
   <xacro:robotiq_arg2f_85 prefix=""/>

File: robotiq_2f_85_description/urdf/robotiq_arg2f_85_model_macro.xacro (robot description, xacro)
@@ -147,5 +147,5 @@
       <child link="${prefix}${fingerprefix}_inner_finger" />
       <axis xyz="1 0 0" />
-      <limit lower="0" upper="0.8757" velocity="2.0" effort="1000" />
+      <limit lower="-0.8757" upper="0.8757" velocity="2.0" effort="1000" />
       <mimic joint="${prefix}finger_joint" multiplier="-1" offset="0" />
     </joint>

File: robotiq_3f_description/urdf/robotiq-3f-gripper_articulated_macro.xacro (robot description, xacro)
@@ -30,5 +30,5 @@
 			</collision>
 		</link>
-		<link name="${prefix}tool0"/>
+		<!-- <link name="${prefix}tool0"/> -->
         <inertial>
             <origin xyz="0 0 0" rpy="0 0 0"/>
@@ -58,9 +58,9 @@
 			<origin xyz="0.0455 0.0214 0" rpy="0 0 1.57"/>
 		</joint>
-		<joint name="${prefix}palm_tool0" type="fixed">
+		<!-- <joint name="${prefix}palm_tool0" type="fixed">
 			<parent link="${prefix}palm"/>
 			<child link="${prefix}tool0"/>
 			<origin xyz="0.0 0.0875 0.0" rpy="0 0 1.5707"/>
-		</joint>
+		</joint> -->
 		<!-- end of joint list -->
 	</xacro:macro>
