Commit message: update

File: robotiq_3f_description/urdf/robotiq-3f-gripper_articulated_macro.xacro (robot description, xacro)
@@ -51,4 +51,5 @@
 			<origin xyz="-0.0455 0.0214 -0.036" rpy="0 3.1416 -1.57"/>
 			<limit lower="-0.192" upper="0.1784" effort="100" velocity="100"/>
+			<mimic joint="${prefix}palm_finger_1_joint" multiplier="-1" offset="0" />
 		</joint>
 		<joint name="${prefix}palm_finger_middle_joint" type="fixed">

File: robotiq_3f_description/urdf/robotiq-3f-gripper_finger_articulated_macro.xacro (robot description, xacro)
@@ -116,4 +116,5 @@
 			<origin xyz="0.050 -.028 0" rpy="0 0 -0.52"/>
 			<limit lower="0.0" upper="1.5708" effort="100" velocity="100"/>
+			<mimic joint="${prefix}joint_1" multiplier="1.5" offset="0" />
 		</joint>
 		<joint name="${prefix}joint_3" type="revolute">
@@ -123,4 +124,5 @@
 			<origin xyz="0.039 0 0" rpy="0 0 0"/>
 			<limit lower="-1.2217" upper="-0.0523" effort="100" velocity="100"/>
+			<mimic joint="${prefix}joint_1" multiplier="-1" offset="0" />
 		</joint>
 		<!-- end of joint list -->
