Commit message: update

File: conveyor_gripper_description/urdf/conveyor_gripper.xacro (robot description, xacro)
@@ -23,3 +23,26 @@
     <child link="conveyor_gripper" />
   </joint>
+  <!-- end effect point -->
+  <joint name="end_effect_point" type="fixed">
+    <origin rpy="0 0 0" xyz="0 -0.050 0.200"/>
+    <parent link="tcp"/>
+    <child link="end_effect_point"/>
+  </joint>
+  <!-- end effect point -->
+  <link name="end_effect_point">
+    <visual>
+      <origin rpy="0 0 0" xyz="0 0 0"/>
+      <geometry>
+        <box size="0.01 0.01 0.01"/>
+      </geometry>
+      <material name="">
+        <color rgba="0.8 0.0 0.0 1.0"/>
+      </material>
+    </visual>
+    <inertial>
+      <origin rpy="0 0 0" xyz="0.0 0.0 0.0"/>
+      <mass value="0.001"/>
+      <inertia ixx="1.0e-06" ixy="0.0" ixz="0.0" iyy="1.0e-06" iyz="0.0" izz="1.0e-06"/>
+    </inertial>
+  </link>
 </robot>
